File: pcb/pcb_topsulin.kicad_pcb (KiCad board)
At the start: 2 copper layers, 91 x 30 mm, 35 parts, among them J1 Conn_01x01_Male, J10 Conn_01x01_Male, J11 Conn_01x01_Male, J12 Conn_01x01_Male, J13 Conn_01x01_Male, J2 Conn_01x01_Male, J3 Conn_01x24, J4 Conn_01x01_Male, J5 Conn_01x01_Male, J6 Conn_01x01_Male, J7 Conn_01x01_Male, J8 Conn_01x01_Male, J9 Conn_01x01_Male, Q1 Q_NMOS_GSD, SW1 Rotary_Encoder_Switch, U1 nRF51822_module_waveshare

Commit message: add pcb
Parts:
- BT1: footprint Battery:BatteryHolder_MPD_BC2003_1x2032 -> Battery:BatteryHolder_Keystone_1058_1x2032
- moved BT1 4.53 mm to (172.5, 99.1), turned to 55 degrees
- moved J6 2.54 mm to (167.1, 86.4)
- moved J9 2.54 mm to (169.7, 86.4)
Routing:
- net C: track 183.4 -> 121.0 mm, vias 5 -> 10
- net +3V3: track 112.6 -> 94.7 mm
- net Net-(J8-Pad1): track 13.0 -> 14.5 mm
- net A: vias 0 -> 1
