File: pcb/pcb_topsulin.sch (KiCad schematic (older format))
At the start: 35 parts, among them J1 Conn_01x01_Male, J10 Conn_01x01_Male, J11 Conn_01x01_Male, J12 Conn_01x01_Male, J13 Conn_01x01_Male, J2 Conn_01x01_Male, J3 Conn_01x24, J4 Conn_01x01_Male, J5 Conn_01x01_Male, J6 Conn_01x01_Male, J7 Conn_01x01_Male, J8 Conn_01x01_Male, J9 Conn_01x01_Male, Q1 Q_NMOS_GSD, SW1 Rotary_Encoder_Switch, U1 nRF51822_module_waveshare

Commit message: Switch to linux
Parts:
- removed U1: nRF51822_module_waveshare, pcb_topsulin:nRF51822_module_waveshare_footprint, symbol topsulin_library:nRF51822_module_waveshare
- added U1: topsulin_topsulin_library_nRF51822_module_wavesha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, symbol topsulin:topsulin_topsulin_topsulin_topsulin_library_nRF51822_module_waveshare
Changed lines of the file:
@@
 EESchema Schematic File Version 4
 LIBS:pcb_topsulin-cache
-EELAYER 26 0
+EELAYER 29 0
 EELAYER END
 $Descr A4 11693 8268
@@
 Comment4 ""
 $EndDescr
-$Comp
-L topsulin_library:nRF51822_module_waveshare U1
-U 1 1 5BCF52CE
-P 2050 1800
-F 0 "U1" H 2050 2865 50  0000 C CNN
-F 1 "nRF51822_module_waveshare" H 2050 2774 50  0000 C CNN
-F 2 "pcb_topsulin:nRF51822_module_waveshare_footprint" H 2050 1800 50  0001 C CNN
-F 3 "" H 2050 1800 50  0001 C CNN
-	1    2050 1800
-	1    0    0    -1
-$EndComp
 Wire Wire Line
 	1350 1100 1100 1100
@@
 Wire Wire Line
 	1650 5200 1850 5200
+$Comp
+L topsulin:topsulin_topsulin_topsulin_topsulin_library_nRF51822_module_waveshare U1
+U 1 1 5CD142A6
+P 2050 1800
+F 0 "U1" H 2050 2915 50  0000 C CNN
+F 1 "topsulin_topsulin_library_nRF51822_module_waveshare" H 2050 2824 50  0000 C CNN
+F 2 "" H 2050 1800 50  0001 C CNN
+F 3 "" H 2050 1800 50  0001 C CNN
+	1    2050 1800
+	1    0    0    -1
+$EndComp
 $EndSCHEMATC

Commit message: add pcb
Parts:
- BT1: footprint Battery:BatteryHolder_MPD_BC2003_1x2032 -> Battery:BatteryHolder_Keystone_1058_1x2032
- J3: footprint kicad_libs:e-paper-2in13-flex-2 -> topsulin:e-paper-2in13-flex
- U1: footprint (none) -> topsulin:nRF51822_module_waveshare_footprint; symbol topsulin:topsulin_topsulin_topsulin_topsulin_library_nRF51822_module_waveshare -> topsulin:topsulin_topsulin_topsulin_topsulin_topsulin_topsulin_topsulin_topsulin_topsulin_topsulin_library_nRF51822_mod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
Changed lines of the file:
@@
 F 0 "J3" H 10580 1792 50  0000 L CNN
 F 1 "Conn_01x24" H 10580 1701 50  0000 L CNN
-F 2 "kicad_libs:e-paper-2in13-flex-2" H 10500 1800 50  0001 C CNN
+F 2 "topsulin:e-paper-2in13-flex" H 10500 1800 50  0001 C CNN
 F 3 "~" H 10500 1800 50  0001 C CNN
 	1    10500 1800
@@
 F 0 "BT1" H 9168 4596 50  0000 L CNN
 F 1 "Battery_Cell" H 9168 4505 50  0000 L CNN
-F 2 "Battery:BatteryHolder_MPD_BC2003_1x2032" V 9050 4560 50  0001 C CNN
+F 2 "Battery:BatteryHolder_Keystone_1058_1x2032" V 9050 4560 50  0001 C CNN
 F 3 "~" V 9050 4560 50  0001 C CNN
 	1    9050 4500
@@
 	1650 5200 1850 5200
 $Comp
-L topsulin:topsulin_topsulin_topsulin_topsulin_library_nRF51822_module_waveshare U1
+L topsulin:topsulin_topsulin_topsulin_topsulin_topsulin_topsulin_topsulin_topsulin_topsulin_topsulin_library_nRF51822_module_waveshare U1
 U 1 1 5CD142A6
 P 2050 1800
 F 0 "U1" H 2050 2915 50  0000 C CNN
 F 1 "topsulin_topsulin_library_nRF51822_module_waveshare" H 2050 2824 50  0000 C CNN
-F 2 "" H 2050 1800 50  0001 C CNN
+F 2 "topsulin:nRF51822_module_waveshare_footprint" H 2050 1800 50  0001 C CNN
 F 3 "" H 2050 1800 50  0001 C CNN
 	1    2050 1800
